File: eagle/atmega.sch (EAGLE design)
At the start: 65 parts, among them IC1 TO 5V, IC2 LM339D, Q2 16MHz, U1 ATMEGA328P-AU

Commit message: Podłączenie wszystkiego zakończone, wystarczy tylko obawić się nad estetyką
Parts:
- removed ZWORKA: (no value), rcl:R-EU_0204/5
- R11: value 220 -> 220R
Connections:
- removed net 7.4V: C3.2, IC1.IN, VOLTAGE.1
- removed net N$31: C6.-, C9.1
- removed net RESET3: R21.1, ZWORKA.2
- new net 5: R8.2
- new net 55: R7.2
- new net 555: R2.2
- new net 5555: R5.2
- new net N$12: U$4.C, U$4.EMI
- new net N$14: U$3.C, U$3.EMI
- new net N$15: U$5.C, U$5.EMI
- new net N$4: U$2.C, U$2.EMI
- net GND: now also C6.-, C9.1, U1.GND_3; no longer U$2.C, U$2.EMI, U$3.C, U$3.EMI, U$4.C, U$4.EMI, U$5.C, U$5.EMI, U1.GND
- net KO1: now also U1.PD2; no longer U1.PD4
- net KO2: now also U1.PD1; no longer U1.PD3
- net KO3: now also U1.PD4; no longer U1.PD1
- net KO4: now also U1.PD3; no longer U1.PD2
- net RESET1: now also R21.1; no longer ZWORKA.1
- net VCC: no longer R2.2, R5.2, R7.2, R8.2
- net VZ: now also C3.2, IC1.IN, VOLTAGE.1
Other:
- note added: "GND"
- note added: "VCC"
- moved on the sheet: IC2A, IC2B, IC2C, IC2D, LED1, LED3, LED4, LED5, R10, R12, R13, R14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
